Commit message: Answer all 17 masterplan2 comments; fix path lookahead, add grid curriculum
Research turned up a result that reverses my own previous recommendation, so
that goes first.

Margolis et al., "Rapid Locomotion via RL" (RSS 2022, 3.9 m/s on Mini Cheetah)
ablate exactly the design I proposed two commits ago as a simplification:
"In the absence of any curriculum, no useful locomotion behavior is learned,
even at low speeds" -- the robot jitters in place, because uniform sampling from
a wide command range is mostly commands too hard to collect reward from. E3 is
therefore a real gamble, not a safe simplification, and its docstring now says
so. The same paper explains WHY a scalar curriculum is not enough: their
curriculum is a grid over (v_x, omega_z) because high linear and high angular
velocity together are much harder than either alone, roughly omega ~ 1/v at the
feasibility boundary. A scalar level cannot represent that boundary -- which is
the reviewer's own point about translation/rotation coupling, independently
arrived at.

Code:

  lookahead was dead code. _reroll_paths sampled self.lookahead from
  [0.5, 3.0] and NOTHING ever read it. The goal was anchored on the robot and
  then ran away, i.e. a pacer, not a lookahead -- the smoke test measured gap
  median 0.41 m, below the configured 0.5 m minimum. That matters because
  constellation is exp(-w d^2), so with the goal sitting on the robot the reward
  is at its maximum and its gradient is ~0: the mechanism built to demand speed
  was flattening the gradient exactly where the robot was. Now clamped by three
  constraints -- pace (creates the demand), floor (keeps it a lookahead), leash
  (keeps the gradient alive when behind). Verified numerically: a robot slower
  than pace parks at the leash, a faster one pins at the floor and drags the
  carrot faster than commanded, which is what lets achieved speed reveal the
  physical ceiling rather than the commanded one.

  Grid-adaptive curriculum over (speed x curvature). On a path omega = v*kappa,
  so this IS Margolis's (v, omega) grid reparameterised, and it trains the
  coupling explicitly. Curvature is commanded through path size. Off by default.

  Serpentine path (shape 5): translation advances monotonically while curvature
  flips sign every half period -- the canonical coupling stress case.

  path_lag = max(gap - lookahead_min, 0). Goal distance can never reach zero in
  path mode by construction, so distance was never the tracking error.

  Arms rebuilt at 90 deg, not 80. The splay widened the ego footprint by 82 mm,
  working against the reason the arms are pinned at all. Ego half-width
  0.396 -> 0.154 m, arm I_zz -61%, I_xx -62%. While doing this the URDF turned
  out to make the requested elbow tuck impossible: Elbow_Pitch's axis [0,1,0] is
  PARALLEL to the forearm offset [0,0.044,0] (a twist, not a bend) and Elbow_Yaw
  sits distal to the forearm, so neither elbow joint moves the 0.762 kg forearm
  mass at all. Only the shoulder can reposition the arm, so the rearward tuck
  uses Shoulder_Pitch +25 deg -> hand 74 mm behind the hip, ego width unchanged.

  Instrumentation audit found 3 of 8 v7 intents had no measurement: curriculum
  progress, joint-limit occupancy, and left/right symmetry. A zero protection
  penalty was ambiguous between "well inside limits" and "term switched off",
  and we switched the symmetry loss on without any way to check whether
  left/right actually became symmetric. All three now exported.

Docs: every comment answered inline with evidence, including the two
explain-it-simply requests. Corrected two stale claims -- the goal_reached
angular term and the stress:jitter mode were both already implemented and
running, but the doc still listed them as pending.

Co-Authored-By: Claude <noreply@anthropic.com>

File: htwk-gym/resources/K1/K1_locomotion_armsdown.urdf (robot description, URDF)
Before this commit: robot K1, 23 links, 22 joints
Joints:
- joint ALeft_Shoulder_Pitch: origin xyz=0 0.077 0.1845 rpy=0 0 0 -> xyz=0 0.077 0.1845 rpy=0.00000 0.43633 0.00000
- joint ARight_Shoulder_Pitch: origin xyz=0 -0.077 0.1845 rpy=0 0 0 -> xyz=0 -0.077 0.1845 rpy=0.00000 0.43633 0.00000
- joint Left_Shoulder_Roll: origin xyz=0.0025 0.068 -0.0135 rpy=-1.39626 0 0 -> xyz=0.0025 0.068 -0.0135 rpy=-1.57080 0.00000 0.00000
- joint Right_Shoulder_Roll: origin xyz=0.0025 -0.068 -0.0135 rpy=1.39626 0 0 -> xyz=0.0025 -0.068 -0.0135 rpy=1.57080 0.00000 0.00000
