Commit message: Implement the arm swing properly; fix symmetry telemetry that never shipped
Three corrections, all of them mine.

The elbows CAN move the hand, and I said twice that they could not. That
conclusion came from checking the T-pose only. Once the arm hangs, the axes
change role: Elbow_Pitch's [0,1,0] points straight down and is therefore a yaw
that aims the bend plane, and Elbow_Yaw's axis becomes horizontal and is the
actual bend -- exactly the "yaw it inward, bend the elbow a little" that was
asked for, twice. Solved by FK within the joint limits: Shoulder_Roll -/+90,
Elbow_Pitch +119.2, Elbow_Yaw -/+90.5 puts the hand 3.1 cm behind the hip with
ego half-width 0.146 m and arm I_zz down 69% (better than the 80-degree splay it
replaces on every axis). Mirror convention verified: under y -> -y, Rx and Rz
flip and Ry is preserved, which reproduces the left and right hands at exactly
+-0.067 m.

The dynamic swing is implemented rather than deferred again. Four elbows become
revolute in K1_locomotion_armswing.urdf and are driven from a closed form, kept
out of the action and observation vectors so num_actions stays 12 and the
observation stays 54 -- E0's weights still load, which is the only reason this
is affordable. That needed two one-line seams in the frozen base
(_dof_targets_from_actions, _obs_dofs) rather than duplicating step(). The
trigger reuses the reward's own parked test instead of a hand-picked speed
cutoff, so "stopped" has one definition in the system, and the pose is blended
over 0.25 s because stepping 2.9 kg of arm would kick the base at every start
and stop. On in G3.

The symmetry metric was worse than "never looked at": it never reached a report.
It was written into env.extras["v7"] and eval_goal_pose read that nowhere, so
all four v7 reports have no such field -- every claim of having added
instrumentation was hollow. Worse, it measured fore-aft only, and the actual
observation was that fore-aft looks fine while the stance sits off-centre with
the right hip yaw pulled inward, which that term cannot express. Now plumbed
through to report.json and measured in the BASE frame (in world frame a turning
robot's left/right difference oscillates with heading and averages to zero
regardless of gait), split into fore-aft, lateral offset, stance width, and
per-joint left/right bias -- bias_Hip_Yaw reads the reported problem directly.

Also adds draw_goal_sequence so G4 can be judged at all: sequential navigation
is about setting up a turn before arriving, which is invisible when the video
shows one goal marker. Banked/active/upcoming goals are colour-coded, written
through inset[..., :3] so it is correct for RGBA camera frames -- the same class
of bug as 5493840.

Co-Authored-By: Claude <noreply@anthropic.com>

File: htwk-gym/resources/K1/K1_locomotion_armswing.urdf (robot description, URDF)
Before this commit: robot K1, 23 links, 22 joints
Joints:
- joint Left_Elbow_Pitch: type fixed -> revolute
- joint Left_Elbow_Yaw: type fixed -> revolute
- joint Right_Elbow_Pitch: type fixed -> revolute
- joint Right_Elbow_Yaw: type fixed -> revolute
